File: rt3050.kicad_pcb (KiCad board)
At the start: 2 copper layers, 90.6 x 35 mm, 60 parts, among them J1 USB, K1 CONN_SERIAL, P1 CONN_JTAG, P2 CONN_RF, P3 CONN_1, P4 CONN_SERIAL2, P5 CONN_SPI, P6 CONN_2, P7 CONN_1, P8 CONN_USB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

Commit message: as sent for r1 to hackvana.
Other:
- board text added: "5DLX"
- board text added: "r1"

Commit message: r2 for fab
Other:
- rule pad_to_mask_clearance: 0.15494 -> 0.2
- board text added: "r2"
- board text removed: "r1"
Changed lines of the file:
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@@
     (mod_text_size 1.524 1.524)
     (mod_text_width 0.3048)
-    (pad_size 0.50038 0.50038)
+    (pad_size 0.41 0.41)
     (pad_drill 0)
-    (pad_to_mask_clearance 0.15494)
+    (pad_to_mask_clearance 0.2)
     (aux_axis_origin 0 0)
     (visible_elements FFFFFF7F)
@@
   (module TFBGA289 (layer Front)
     (at 158.60014 92.09786)
-    (solder_mask_margin 0.01016)
-    (clearance 0.01016)
+    (solder_mask_margin 0.07)
+    (clearance 0.07)
     (fp_text reference U1 (at 0 -9.6012) (layer F.SilkS)
       (effects (font (thickness 0.3048)))
@@
       (net 17 N-000016))
   )
-  (gr_text r1 (at 214.7 81.1) (layer F.SilkS)
+  (gr_text r2 (at 214.7 81.1) (layer F.SilkS)
     (effects (font (size 2.032 1.524) (thickness 0.3048)))
   )
@@
   (segment (start 154.99842 93.69806) (end 154.5971 93.69806) (width 0.29972) (layer Front) (net 1) (status 20))
   (segment (start 154.5971 93.69806) (end 154.5971 94.49816) (width 0.29972) (layer Front) (net 1) (status 30))
-  (segment (start 154.59964 94.49816) (end 154.5971 94.49816) (width 0.50038) (layer Front) (net 1) (status 30))
+  (segment (start 154.59964 94.49816) (end 154.5971 94.49816) (width 0.2032) (layer Front) (net 1) (status 30))
   (segment (start 154.99842 93.69806) (end 154.5971 94.09938) (width 0.29972) (layer Front) (net 1))
   (via (at 154.5971 94.09938) (size 0.29972) (drill 0.20066) (layers Front Back) (net 1))

Commit message: hackvana final
Other:
- board text added: "r3"
- board text removed: "r2"
