File: RT3050RF.sch (KiCad schematic (older format))
At the start: 10 parts, among them P2 CONN_5, U1 RT3050

Commit message: updated component values
Parts:
- C14: value C -> 1uF
Changed lines of the file:
@@
-EESchema Schematic File Version 2  date Tue 02 Sep 2014 05:26:51 BST
+EESchema Schematic File Version 2
 LIBS:power
 LIBS:device
@@
 LIBS:AIC809
 LIBS:rt3050-cache
-EELAYER 25  0
+EELAYER 25 0
 EELAYER END
-$Descr A4 11700 8267
+$Descr A4 11693 8268
 encoding utf-8
 Sheet 2 6
@@
 F 0 "#PWR01" H 4700 3990 20  0001 C CNN
 F 1 "+1.2V" H 4700 3960 30  0000 C CNN
+F 2 "" H 4700 3850 60  0001 C CNN
+F 3 "" H 4700 3850 60  0001 C CNN
 	1    4700 3850
 	1    0    0    -1
@@
 F 0 "#PWR02" H 4700 4360 30  0001 C CNN
 F 1 "+3.3V" H 4700 4510 30  0000 C CNN
+F 2 "" H 4700 4400 60  0001 C CNN
+F 3 "" H 4700 4400 60  0001 C CNN
 	1    4700 4400
 	1    0    0    -1
@@
 F 0 "#PWR03" H 800 3810 30  0001 C CNN
 F 1 "+3.3V" H 800 3960 30  0000 C CNN
+F 2 "" H 800 3850 60  0001 C CNN
+F 3 "" H 800 3850 60  0001 C CNN
 	1    800  3850
 	1    0    0    -1
@@
 F 0 "#PWR04" H 1300 5560 30  0001 C CNN
 F 1 "+3.3V" H 1300 5710 30  0000 C CNN
+F 2 "" H 1300 5600 60  0001 C CNN
+F 3 "" H 1300 5600 60  0001 C CNN
 	1    1300 5600
 	1    0    0    -1
@@
 F 0 "#PWR05" H 4850 3790 20  0001 C CNN
 F 1 "+1.2V" H 4850 3760 30  0000 C CNN
+F 2 "" H 4850 3650 60  0001 C CNN
+F 3 "" H 4850 3650 60  0001 C CNN
 	1    4850 3650
 	1    0    0    -1
@@
 F 0 "P2" V 550 3150 50  0000 C CNN
 F 1 "CONN_5" V 650 3150 50  0000 C CNN
+F 2 "" H 600 3150 60  0001 C CNN
+F 3 "" H 600 3150 60  0001 C CNN
 	1    600  3150
 	-1   0    0    1
@@
 F 0 "C16" H 5650 6550 50  0000 L CNN
 F 1 "C" H 5650 6350 50  0000 L CNN
+F 2 "" H 5600 6450 60  0001 C CNN
+F 3 "" H 5600 6450 60  0001 C CNN
 	1    5600 6450
 	1    0    0    -1
@@
 F 0 "#PWR06" H 5950 6700 30  0001 C CNN
 F 1 "GND" H 5950 6630 30  0001 C CNN
+F 2 "" H 5950 6700 60  0001 C CNN
+F 3 "" H 5950 6700 60  0001 C CNN
 	1    5950 6700
 	1    0    0    -1
@@
 F 0 "C17" H 6000 6550 50  0000 L CNN
 F 1 "C" H 6000 6350 50  0000 L CNN
+F 2 "" H 5950 6450 60  0001 C CNN
+F 3 "" H 5950 6450 60  0001 C CNN
 	1    5950 6450
 	1    0    0    -1
@@
 F 0 "#PWR07" H 650 4490 20  0001 C CNN
 F 1 "+1.2V" H 650 4460 30  0000 C CNN
+F 2 "" H 650 4350 60  0001 C CNN
+F 3 "" H 650 4350 60  0001 C CNN
 	1    650  4350
 	1    0    0    -1
@@
 F 0 "#PWR08" H 5550 4190 20  0001 C CNN
 F 1 "+1.2V" H 5550 4160 30  0000 C CNN
+F 2 "" H 5550 4050 60  0001 C CNN
+F 3 "" H 5550 4050 60  0001 C CNN
 	1    5550 4050
 	1    0    0    -1
@@
 F 0 "#PWR09" H 5100 3290 20  0001 C CNN
 F 1 "+1.2V" H 5100 3260 30  0000 C CNN
+F 2 "" H 5100 3150 60  0001 C CNN
+F 3 "" H 5100 3150 60  0001 C CNN
 	1    5100 3150
 	1    0    0    -1
@@
 F 0 "#PWR010" H 1000 4340 20  0001 C CNN
 F 1 "+1.2V" H 1000 4310 30  0000 C CNN
+F 2 "" H 1000 4200 60  0001 C CNN
+F 3 "" H 1000 4200 60  0001 C CNN
 	1    1000 4200
 	1    0    0    -1
@@
 F 0 "#PWR011" H 5400 6150 30  0001 C CNN
 F 1 "GND" H 5400 6080 30  0001 C CNN
+F 2 "" H 5400 6150 60  0001 C CNN
+F 3 "" H 5400 6150 60  0001 C CNN
 	1    5400 6150
 	1    0    0    -1
@@
 P 5400 5850
 F 0 "C14" H 5450 5950 50  0000 L CNN
-F 1 "C" H 5450 5750 50  0000 L CNN
+F 1 "1uF" H 5450 5750 50  0000 L CNN
+F 2 "" H 5400 5850 60  0001 C CNN
+F 3 "" H 5400 5850 60  0001 C CNN
 	1    5400 5850
 	1    0    0    -1
@@
 F 0 "C11" H 4900 5650 50  0000 L CNN
 F 1 "C" H 4900 5450 50  0000 L CNN
+F 2 "" H 4850 5550 60  0001 C CNN
+F 3 "" H 4850 5550 60  0001 C CNN
 	1    4850 5550
 	1    0    0    -1
@@
 F 0 "C9" H 4850 6300 50  0000 L CNN
 F 1 "C" H 4850 6100 50  0000 L CNN
+F 2 "" H 4800 6200 60  0001 C CNN
+F 3 "" H 4800 6200 60  0001 C CNN
 	1    4800 6200
 	1    0    0    -1
@@
 F 0 "#PWR012" H 550 5140 20  0001 C CNN
 F 1 "+1.2V" H 550 5110 30  0000 C CNN
+F 2 "" H 550 5000 60  0001 C CNN
+F 3 "" H 550 5000 60  0001 C CNN
 	1    550  5000
 	1    0    0    -1
@@
 F 0 "#PWR013" H 950 6700 30  0001 C CNN
 F 1 "GND" H 950 6630 30  0001 C CNN
+F 2 "" H 950 6700 60  0001 C CNN
+F 3 "" H 950 6700 60  0001 C CNN
 	1    950  6700
 	1    0    0    -1
@@
 F 0 "R11" V 830 6250 50  0000 C CNN
 F 1 "R" V 750 6250 50  0000 C CNN
+F 2 "" H 750 6250 60  0001 C CNN
+F 3 "" H 750 6250 60  0001 C CNN
 	1    750  6250
 	1    0    0    -1
@@
 F 0 "C8" H 1200 6350 50  0000 L CNN
 F 1 "C" H 1200 6150 50  0000 L CNN
+F 2 "" H 1150 6250 60  0001 C CNN
+F 3 "" H 1150 6250 60  0001 C CNN
 	1    1150 6250
 	1    0    0    -1
@@
 F 0 "#PWR014" H 5200 5400 30  0001 C CNN
 F 1 "GND" H 5200 5330 30  0001 C CNN
+F 2 "" H 5200 5400 60  0001 C CNN
+F 3 "" H 5200 5400 60  0001 C CNN
 	1    5200 5400
 	1    0    0    -1
@@
 F 0 "C13" H 5250 5200 50  0000 L CNN
 F 1 "C" H 5250 5000 50  0000 L CNN
+F 2 "" H 5200 5100 60  0001 C CNN
+F 3 "" H 5200 5100 60  0001 C CNN
 	1    5200 5100
 	1    0    0    -1
@@
 F 0 "U1" H 3050 -400 60  0000 C CNN
 F 1 "RT3050" H 2950 8950 60  0000 C CNN
+F 2 "" H 3050 5050 60  0001 C CNN
+F 3 "" H 3050 5050 60  0001 C CNN
 	5    3050 5050
 	1    0    0    -1
@@
 F 0 "#PWR015" H 5100 3540 20  0001 C CNN
 F 1 "+1.2V" H 5100 3510 30  0000 C CNN
+F 2 "" H 5100 3400 60  0001 C CNN
+F 3 "" H 5100 3400 60  0001 C CNN
 	1    5100 3400
 	1    0    0    -1
