File: RT3050main.sch (KiCad schematic (older format))
At the start: 14 parts, among them K1 CONN_SERIAL, P1 CONN_JTAG, P4 CONN_SERIAL2, P5 CONN_SPI, P6 CONN_2, P7 CONN_1, P8 CONN_USB, U1 RT3050, U6 AIC809, X1 XO

Commit message: updated component values
Parts:
- C2: value C -> 40pF
- R: renamed from C1; value C -> 0; symbol C -> R
Connections:
- net at C2.1, X1.3 (OUTPUT): no longer R.1
- net at U1.C7 (PLL_X2): no longer R.2
Changed lines of the file:
@@
-EESchema Schematic File Version 2  date Tue 02 Sep 2014 05:26:51 BST
+EESchema Schematic File Version 2
 LIBS:power
 LIBS:device
@@
 LIBS:AIC809
 LIBS:rt3050-cache
-EELAYER 25  0
+EELAYER 25 0
 EELAYER END
-$Descr A4 11700 8267
+$Descr A4 11693 8268
 encoding utf-8
 Sheet 6 6
@@
 F 0 "P7" H 5380 4600 40  0000 L CNN
 F 1 "CONN_1" H 5300 4655 30  0001 C CNN
+F 2 "" H 5300 4600 60  0001 C CNN
+F 3 "" H 5300 4600 60  0001 C CNN
 	1    5300 4600
 	1    0    0    -1
@@
 F 0 "P6" V 5100 4100 40  0000 C CNN
 F 1 "CONN_2" V 5200 4100 40  0000 C CNN
+F 2 "" H 5150 4100 60  0001 C CNN
+F 3 "" H 5150 4100 60  0001 C CNN
 	1    5150 4100
 	1    0    0    -1
@@
 F 0 "P5" V 1000 2950 50  0000 C CNN
 F 1 "CONN_SPI" V 1100 2950 50  0000 C CNN
+F 2 "" H 1050 2950 60  0001 C CNN
+F 3 "" H 1050 2950 60  0001 C CNN
 	1    1050 2950
 	-1   0    0    1
@@
 F 0 "P8" V 5650 6750 50  0000 C CNN
 F 1 "CONN_USB" V 5750 6750 50  0000 C CNN
+F 2 "" H 5700 6750 60  0001 C CNN
+F 3 "" H 5700 6750 60  0001 C CNN
 	1    5700 6750
 	1    0    0    -1
@@
 F 0 "#PWR044" H 5400 5550 30  0001 C CNN
 F 1 "GND" H 5400 5480 30  0001 C CNN
+F 2 "" H 5400 5550 60  0001 C CNN
+F 3 "" H 5400 5550 60  0001 C CNN
 	1    5400 5550
 	1    0    0    -1
@@
 F 0 "R20" V 5480 5250 50  0000 C CNN
 F 1 "R" V 5400 5250 50  0000 C CNN
+F 2 "" H 5400 5250 60  0001 C CNN
+F 3 "" H 5400 5250 60  0001 C CNN
 	1    5400 5250
 	1    0    0    -1
@@
 F 0 "D1" H 5100 5100 50  0000 C CNN
 F 1 "LED" H 5100 4900 50  0000 C CNN
+F 2 "" H 5100 5000 60  0001 C CNN
+F 3 "" H 5100 5000 60  0001 C CNN
 	1    5100 5000
 	1    0    0    -1
@@
 F 0 "P4" V 700 1650 60  0000 C CNN
 F 1 "CONN_SERIAL2" V 800 1650 60  0000 C CNN
+F 2 "" H 750 1650 60  0001 C CNN
+F 3 "" H 750 1650 60  0001 C CNN
 	1    750  1650
 	-1   0    0    1
@@
 F 0 "#PWR045" H 5400 3540 20  0001 C CNN
 F 1 "+1.2V" H 5400 3510 30  0000 C CNN
+F 2 "" H 5400 3400 60  0001 C CNN
+F 3 "" H 5400 3400 60  0001 C CNN
 	1    5400 3400
 	1    0    0    -1
@@
 F 0 "#PWR046" H 7350 5700 30  0001 C CNN
 F 1 "GND" H 7350 5630 30  0001 C CNN
+F 2 "" H 7350 5700 60  0001 C CNN
+F 3 "" H 7350 5700 60  0001 C CNN
 	1    7350 5700
 	1    0    0    -1
@@
 F 0 "#PWR047" H 7100 5010 30  0001 C CNN
 F 1 "+3.3V" H 7100 5160 30  0000 C CNN
+F 2 "" H 7100 5050 60  0001 C CNN
+F 3 "" H 7100 5050 60  0001 C CNN
 	1    7100 5050
 	1    0    0    -1
@@
 F 0 "U6" H 7900 4500 60  0000 C CNN
 F 1 "AIC809" H 7900 5750 60  0000 C CNN
+F 2 "" H 7900 5150 60  0001 C CNN
+F 3 "" H 7900 5150 60  0001 C CNN
 	1    7900 5150
 	1    0    0    -1
@@
 F 0 "#PWR048" H 6700 1550 30  0001 C CNN
 F 1 "GND" H 6700 1480 30  0001 C CNN
+F 2 "" H 6700 1550 60  0001 C CNN
+F 3 "" H 6700 1550 60  0001 C CNN
 	1    6700 1550
 	1    0    0    -1
@@
 F 0 "P1" V 7000 1100 60  0000 C CNN
 F 1 "CONN_JTAG" V 7100 1100 60  0000 C CNN
+F 2 "" H 7050 1100 60  0001 C CNN
+F 3 "" H 7050 1100 60  0001 C CNN
 	1    7050 1100
 	1    0    0    -1
@@
 F 0 "#PWR049" H 6150 2050 30  0001 C CNN
 F 1 "GND" H 6150 1980 30  0001 C CNN
+F 2 "" H 6150 2050 60  0001 C CNN
+F 3 "" H 6150 2050 60  0001 C CNN
 	1    6150 2050
 	1    0    0    -1
@@
 F 0 "K1" V 6850 2100 50  0000 C CNN
 F 1 "CONN_SERIAL" V 6950 2100 40  0000 C CNN
+F 2 "" H 6900 2100 60  0001 C CNN
+F 3 "" H 6900 2100 60  0001 C CNN
 	1    6900 2100
 	1    0    0    -1
 $EndComp
 $Comp
-L C C1
+L R R
 U 1 1 53F0A047
 P 5600 2950
-F 0 "C1" H 5650 3050 50  0000 L CNN
-F 1 "C" H 5650 2850 50  0000 L CNN
+F 0 "R" H 5650 3050 50  0000 L CNN
+F 1 "0" H 5650 2850 50  0000 L CNN
+F 2 "" H 5600 2950 60  0001 C CNN
+F 3 "" H 5600 2950 60  0001 C CNN
 	1    5600 2950
 	0    1    1    0
@@
 P 6150 3150
 F 0 "C2" H 6200 3250 50  0000 L CNN
-F 1 "C" H 6200 3050 50  0000 L CNN
+F 1 "40pF" H 6200 3050 50  0000 L CNN
+F 2 "" H 6150 3150 60  0001 C CNN
+F 3 "" H 6150 3150 60  0001 C CNN
 	1    6150 3150
 	1    0    0    -1
@@
 F 0 "#PWR050" H 6400 3600 30  0001 C CNN
 F 1 "GND" H 6400 3530 30  0001 C CNN
+F 2 "" H 6400 3600 60  0001 C CNN
+F 3 "" H 6400 3600 60  0001 C CNN
 	1    6400 3600
 	1    0    0    -1
@@
 F 0 "U1" H 3350 -1450 60  0000 C CNN
 F 1 "RT3050" H 3250 7900 60  0000 C CNN
+F 2 "" H 3350 4000 60  0001 C CNN
+F 3 "" H 3350 4000 60  0001 C CNN
 	1    3350 4000
 	1    0    0    -1
@@
 F 0 "X1" H 7050 3150 60  0000 C CNN
 F 1 "XO" H 7050 2450 60  0000 C CNN
+F 2 "" H 7050 2800 60  0001 C CNN
+F 3 "" H 7050 2800 60  0001 C CNN
 	1    7050 2800
 	1    0    0    -1
